File: basico.sch (KiCad schematic (older format))
At the start: 8 parts, among them P1 Power, P2 Analog, P3 Analog, P4 Digital, P5 PWM, P6 PWM, P7 Communication

Commit message: Cleanup
Other:
- note added: "Arduino Mega Rev 3 Headers"
- note added: "Poncho Smart RAMPS para EDU-CIAA-NXP\n"
- note removed: "Este diseño puede copiarse para iniciar un poncho simple. \n1) Copiar toda la carpeta "Basico" , renombrando \n la misma al nombre del poncho.\n2) Renombrar los archivos "basico.xxx" manteniendo \n las extensiones pero cambiando a un nombre \n descriptivo del poncho. Evitar acentos, espacios y \n caracteres ascii esxtendidos."
- note removed: "Luego de abrir el nuevo proyecto:\n1)Editar datos del rótulo.\n2)Editar los archivos del subdirectorio "doc".\n2.1) Agregarse en el archivo de licencia.\n2.2) Colocar info mínima del Poncho en el LEEME.txt\n2.3) Colocar info mínima en el CAMBIOS.txt"
- note removed: "Shield for Arduino Mega Rev 3"
Changed lines of the file:
@@
 encoding utf-8
 Sheet 1 1
-Title "Poncho Básico (Editar y colocar el nombre final)"
-Date "2016-08-07"
+Title "Poncho Smart RAMPS para EDU-CIAA-NXP"
+Date "2019-06-11"
 Rev "1.0"
 Comp "Proyecto CIAA - COMPUTADORA INDUSTRIAL ABIERTA ARGENTINA"
 Comment1 "https://github.com/ciaa/Ponchos/tree/master/Basico/doc"
-Comment2 "Autores y Licencia del modelo (Diego Brengi - UNLaM)"
-Comment3 "Autor del poncho (COMPLETAR NOMBRE Y APELLIDO). Ver directorio \"doc\""
+Comment2 "Licencia GPL v3 (Emilio Moretti - UNNOBA)"
+Comment3 "Ing. Moretti Emilio"
 Comment4 ""
 $EndDescr
@@
 	1    0    0    -1
 $EndComp
-Text Notes 2950 7650 0    60   ~ 0
-Luego de abrir el nuevo proyecto:\n1)Editar datos del rótulo.\n2)Editar los archivos del subdirectorio "doc".\n2.1) Agregarse en el archivo de licencia.\n2.2) Colocar info mínima del Poncho en el LEEME.txt\n2.3) Colocar info mínima en el CAMBIOS.txt
 $Comp
 L basico-rescue:Conn_Poncho2P_2x_20x2 XA101
@@
 Ar_AREF
 Text Notes 8375 575  0    60   ~ 0
-Shield for Arduino Mega Rev 3
+Arduino Mega Rev 3 Headers
 Text Notes 9650 1350 0    60   ~ 0
 1
@@
 Wire Notes Line
 	8350 6050 8350 500
-Text Notes 7900 -1300 0    118  ~ 24
+Text Notes 3650 6750 0    118  ~ 24
 http://www.proyecto-ciaa.com.ar/
-Text Notes 7850 -250 0    79   Italic 16
-Este diseño puede copiarse para iniciar un poncho simple. \n1) Copiar toda la carpeta "Basico" , renombrando \n   la misma al nombre del poncho.\n2) Renombrar los archivos "basico.xxx" manteniendo \n    las extensiones pero cambiando a un nombre \n    descriptivo del poncho. Evitar acentos, espacios y \n    caracteres ascii esxtendidos.
 Wire Wire Line
 	9000 5350 9000 5750
@@
 NoConn ~ 1800 1850
 NoConn ~ 1800 1950
+Text Notes 1375 675  0    60   ~ 0
+Poncho Smart RAMPS para EDU-CIAA-NXP\n
 $EndSCHEMATC
